Commit message: Modify URDF to include speed limits

File: fairino_description/urdf/fairino20_v6.urdf (robot description, URDF)
Before this commit: robot fairino20_v6_robot, 7 links, 6 joints
Joints:
- joint j1: limit lower=-3.0543 upper=3.0543 effort=150 velocity=3.15 -> lower=-3.0543 upper=3.0543 effort=150 velocity=0.7853981633974483
- joint j2: limit lower=-4.6251 upper=1.4835 effort=150 velocity=3.15 -> lower=-4.6251 upper=1.4835 effort=150 velocity=0.7853981633974483
- joint j3: limit lower=-2.8274 upper=2.8274 effort=150 velocity=3.15 -> lower=-2.8274 upper=2.8274 effort=150 velocity=0.7853981633974483
- joint j4: limit lower=-4.6251 upper=1.4835 effort=28 velocity=3.2 -> lower=-4.6251 upper=1.4835 effort=28 velocity=0.7853981633974483
- joint j5: limit lower=-3.0543 upper=3.0543 effort=28 velocity=3.2 -> lower=-3.0543 upper=3.0543 effort=28 velocity=0.7853981633974483
- joint j6: limit lower=-3.0543 upper=3.0543 effort=28 velocity=3.2 -> lower=-3.0543 upper=3.0543 effort=28 velocity=0.7853981633974483
